File: PCB/SF.kicad_pcb (KiCad board)
At the start: 2 copper layers, 94.7 x 69.2 mm, 33 parts, among them SW1 SW_Push, SW2 SW_Push, SW3 SW_Push, SW4 SW_Push, SW5 SW_Push, SW6 SW_Push, SW7 SW_Push, SW8 SW_Push, U1 XIAO-RP2040-DIP

Commit message: Add files via upload
Parts:
- D1, D10, D2, D3, D4, D5, D6, D7, D8, D9: value SK6812 -> SK6812MINI
- moved D10 37.7 mm to (106.8, 54.4), turned to 0 degrees
- moved D6 36.3 mm to (87.5, 108.0), turned to 0 degrees
- moved D9 26.1 mm to (127.0, 71.0), turned to 0 degrees
- moved D5 25.1 mm to (62.5, 106.0), turned to 0 degrees
- moved D4 23.2 mm to (45.0, 90.5), turned to 0 degrees
- moved D2 20.0 mm to (57.2, 61.9), turned to 0 degrees
- moved D7 18.2 mm to (123.0, 101.5), turned to 0 degrees
- moved D8 14.4 mm to (131.0, 85.0), turned to 0 degrees
- moved D1 13.9 mm to (69.1, 54.8), turned to 0 degrees
- moved D3 12.5 mm to (45.0, 78.0), turned to 0 degrees
Routing:
- net Net-(D6-DOUT): track 16.5 -> 43.0 mm
- net Net-(D10-DIN): track 46.3 -> 25.3 mm
- net RGB: track 43.7 -> 24.3 mm
- net GND: track 54.5 -> 73.2 mm, vias 2 -> 1
- net Net-(D1-DOUT): track 25.4 -> 11.1 mm, vias 2 -> 0
- net Net-(D8-DOUT): track 29.9 -> 17.0 mm, vias 2 -> 0
- net Net-(D3-DOUT): track 23.6 -> 13.1 mm
- net Net-(D7-DOUT): track 15.2 -> 23.0 mm
- net +5V: track 18.8 -> 24.7 mm
- net Net-(D5-DOUT): track 34.2 -> 29.3 mm
- net Net-(D2-DOUT): track 15.7 -> 18.4 mm, vias 2 -> 0
- net Net-(D4-DOUT): vias 0 -> 2
